Commit message: 更新教师训练环境

File: source/visual_wholebody_isaaclab/visual_wholebody_isaaclab/assets/data/obj_set/sugar_box/model.urdf (robot description, URDF)
Before this commit: robot model.urdf, 1 links, 0 joints
Links:
- link baseLink: geometry collision mesh filename=collision.obj scale=1 1 1; visual box size=0.177 0.093 0.046
